File: pcb/usb-can.kicad_sch (KiCad schematic)
At the start: 54 parts, among them J1 Micro_SD_Card_Det1, J2 Conn_ARM_SWD_TagConnect_TC203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, J3 USB_C_Receptacle_USB2.0_16P, J4 Conn_01x04_MountingPin, J5 Conn_01x04_MountingPin, U1 STM32G473CBTx, U2 TJA1042T-3, U3 SRV05-4, U4 AMS1117-3.3, U5 TPS5430DDA, Y1 16MHz

Commit message: Minimize schematic
Parts:
- removed C15: 10n, Capacitor_SMD:C_0402_1005Metric, symbol Device:C
- removed C16, C17: 22u, Capacitor_SMD:C_1206_3216Metric, symbol Device:C
- removed C18: 220u, Capacitor_SMD:CP_Elec_6.3x5.4, symbol Device:C_Polarized
- removed C19: 1n, Capacitor_SMD:C_0603_1608Metric, symbol Device:C
- removed C6, C8: 100n, Capacitor_SMD:C_0402_1005Metric, symbol Device:C
- removed D2: SS34, Diode_SMD:D_SMA, symbol Device:D_Schottky
- removed H1, H2, H3, H4: MountingHole_Pad, MountingHole:MountingHole_3.2mm_M3_ISO7380_Pad, symbol Mechanical:MountingHole_Pad
- removed J1: Micro_SD_Card_Det1, User_Footprints:SD-CARD, symbol Connector:Micro_SD_Card_Det1
- removed JP1, JP2: SolderJumper_2_Open, Jumper:SolderJumper-2_P1.3mm_Open_RoundedPad1.0x1.5mm, symbol Jumper:SolderJumper_2_Open
- removed L1: 15u, Inductor_SMD:L_Sunlord_MWSA0503S, symbol Device:L
- removed R11, R2, R4, R6: 10k, Resistor_SMD:R_0402_1005Metric, symbol Device:R
- removed R12: 3k3, Resistor_SMD:R_0402_1005Metric, symbol Device:R
- removed R13, R14, R15, R8: 120, Resistor_SMD:R_0603_1608Metric, symbol Device:R
- removed U5: TPS5430DDA, Package_SO:TI_SO-PowerPAD-8_ThermalVias, symbol Regulator_Switching:TPS5430DDA
- added SW2: SW_SPDT, symbol Switch:SW_SPDT
- R1: value 10k -> 120; footprint Resistor_SMD:R_0402_1005Metric -> Resistor_SMD:R_1206_3216Metric; LCSC C25744 -> C17909
- R3: value 10k -> 510; LCSC C25744 -> C25123
Connections:
- net +12V is gone; now on net +5V: J4.1 (Pin_1), J5.1 (Pin_1)
- net +3V3: no longer R1.1, R3.1
- net CANH: now also J4.2 (Pin_2), J5.2 (Pin_2), SW2.1 (A); no longer J4.3 (Pin_3), J5.3 (Pin_3)
- net CANL: now also J4.3 (Pin_3), J5.3 (Pin_3), R1.1; no longer J4.2 (Pin_2), J5.2 (Pin_2)
- net RST: no longer U1.7 (PG10)
- net BOOT0: no longer names the net of U1.45 (PB8)
- net CS: no longer names the net of R1.2
- net CS: now also SW2.2 (B); no longer U1.12 (PA4)
- net DET: no longer names the net of U1.16 (PB0)
- net MISO: no longer names the net of U1.14 (PA6)
- net MOSI renamed LEDG
- net LEDG: now also R3.1
- net SCK: no longer names the net of U1.13 (PA5)
- net SCK: no longer R3.2
- no-connect marks 28 -> 31
Other:
- note removed: "5V Regulator"
- note removed: "MicroSD Card"
- note removed: "Mounting"
- moved on the sheet: C1, C10, C11, C12, C13, C14, C2, C3, C4, C5, C7, C9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

Commit message: Finish rev2
Parts:
- removed R5, R7: 510, Resistor_SMD:R_0402_1005Metric, symbol Device:R
- removed SW2: SW_SPDT, symbol Switch:SW_SPDT
- removed U2: TJA1042T-3, Package_SO:SOIC-8_3.9x4.9mm_P1.27mm, symbol Interface_CAN_LIN:TJA1042T-3
- added D2: GLED, LED_SMD:LED_0603_1608Metric, symbol Device:LED
- added JP1: SolderJumper_2_Open, Jumper:SolderJumper-2_P1.3mm_Open_RoundedPad1.0x1.5mm, symbol Jumper:SolderJumper_2_Open
- added R2, R4: 1k, Resistor_SMD:R_0402_1005Metric, symbol Device:R
- added U2: TJA1044GTK/3, Package_SON:HVSON-8-1EP_3x3mm_P0.65mm_EP1.6x2.4mm, symbol User_Symbols:TJA1044GTK/3
- C7, C9: value 10p -> 12p; LCSC C32949 -> C1547
- D1: value LEDB -> LEDR; LCSC C2986058 -> C2286
- R3: value 510 -> 1k; LCSC C25123 -> C11702
Connections:
- net +3V3: now also U2.5 (VIO)
- net +5V: now also U2.3 (VCC)
- net CANH: now also J4.3 (Pin_3), J5.3 (Pin_3), R1.1, U2.7 (CANH); no longer J4.2 (Pin_2), J5.2 (Pin_2)
- net CANL: now also J4.2 (Pin_2), J5.2 (Pin_2), JP1.1 (A), U2.6 (CANL); no longer J4.3 (Pin_3), J5.3 (Pin_3), R1.1
- net CNRX: now also U1.45 (PB8), U2.4 (RXD); no longer U1.26 (PB12)
- net CNTX: now also U1.46 (PB9), U2.1 (TXD); no longer U1.27 (PB13)
- net GND: now also D2.1 (K), U2.2 (GND), U2.8 (STB), U2.9 (EPAD)
- net LEDG: now also U1.12 (PA4); no longer U1.15 (PA7)
- net XTALI: now also C7.2, Y1.1
- net XTALO: now also R2.2; no longer C7.2, Y1.1
- net XTALR: now also R2.1
- net at R1.2: now also JP1.2 (B)
- net at D1.2 (A): now also R4.2
- net LEDR: now reaches U1.10 (PA2)
- net LEDR: now also R4.1
- net at R3.2: now also D2.2 (A)
- net LEDB: no longer names the net of U1.30 (PA8)
- net RST: no longer names the net of J2.3 (~{RESET})
- net SWO: no longer names the net of J2.6 (SWO)
- net SWO: no longer U1.40 (PB3)
- no-connect marks 31 -> 32
Other:
- moved on the sheet: C1, C2, C3, C4, C5, R1, U1
